Commit message: fix gripper macro not transformed

File: workspace/noetic_src/ur_pick_and_place/urdf/ur5/custom_ur5.xacro (robot description, xacro)
@@ -10,8 +10,14 @@
   <!-- robotiq 2f-85 -->
   <xacro:robotiq_arg2f_85 prefix=""/>
+  <link name="world" />
+  <joint name="world_joint" type="fixed">
+    <parent link="world" />
+    <child link = "base_link" />
+    <origin xyz="0.0 0.0 0.0" rpy="0.0 0.0 0.0" />
+  </joint>
   <joint name="eef_gripper_joint" type="fixed">
-    <parent link="wrist_3_link"/>
+    <parent link="flange"/>
     <child link="robotiq_arg2f_base_link"/>
-    <origin xyz="0 0 0" rpy="0.0 0.0 0.0"/>
+    <origin xyz="0 0 0" rpy="0.0 ${pi/2} 0.0"/>
   </joint>
 </robot>

Commit message: Update TODO:  create nodes for performing pick-and-place

File: workspace/noetic_src/ur_pick_and_place/urdf/ur5/custom_ur5.xacro (robot description, xacro)
@@ -16,5 +16,5 @@
     <origin xyz="0.0 0.0 0.0" rpy="0.0 0.0 0.0" />
   </joint>
-  <joint name="eef_gripper_joint" type="fixed">
+  <joint name="ee_gripper_joint" type="fixed">
     <parent link="flange"/>
     <child link="robotiq_arg2f_base_link"/>

Commit message: chore: update moveit config reference

File: workspace/noetic_src/ur_pick_and_place/urdf/ur5/custom_ur5.xacro (robot description, xacro)
@@ -10,10 +10,10 @@
   <!-- robotiq 2f-85 -->
   <xacro:robotiq_arg2f_85 prefix=""/>
-  <link name="world" />
+  <!-- <link name="world" />
   <joint name="world_joint" type="fixed">
     <parent link="world" />
     <child link = "base_link" />
     <origin xyz="0.0 0.0 0.0" rpy="0.0 0.0 0.0" />
-  </joint>
+  </joint> -->
   <joint name="ee_gripper_joint" type="fixed">
     <parent link="flange"/>

Commit message: update custom moveit configuration

File: workspace/noetic_src/ur_pick_and_place/urdf/ur5/custom_ur5.xacro (robot description, xacro)
@@ -10,10 +10,10 @@
   <!-- robotiq 2f-85 -->
   <xacro:robotiq_arg2f_85 prefix=""/>
-  <!-- <link name="world" />
+  <link name="world" />
   <joint name="world_joint" type="fixed">
     <parent link="world" />
     <child link = "base_link" />
     <origin xyz="0.0 0.0 0.0" rpy="0.0 0.0 0.0" />
-  </joint> -->
+  </joint>
   <joint name="ee_gripper_joint" type="fixed">
     <parent link="flange"/>

Commit message: add realsense d455 to custom robot urdf

File: workspace/noetic_src/ur_pick_and_place/urdf/ur5/custom_ur5.xacro (robot description, xacro)
@@ -1,8 +1,11 @@
 <?xml version="1.0"?>
 <robot xmlns:xacro="http://wiki.ros.org/xacro" name="workcell">
+  <xacro:arg name="use_nominal_extrinsics" default="false"/>
   <!-- import ur5 -->
   <xacro:include filename="$(find ur_pick_and_place)/urdf/ur5/ur5_macro.xacro"/>
   <!-- import robotiq 2f-85 -->
   <xacro:include filename="$(find ur_pick_and_place)/urdf/gripper2f85/robotiq_arg2f_85_model_macro.xacro"/>
+  <!-- import realsense d455 -->
+  <xacro:include filename="$(find ur_pick_and_place)/urdf/realsensed455/_d455.urdf.xacro" />
   <!-- parameters -->
   <!-- ur5 -->
@@ -10,4 +13,9 @@
   <!-- robotiq 2f-85 -->
   <xacro:robotiq_arg2f_85 prefix=""/>
+  <!-- realsense d455 -->
+  <xacro:sensor_d455 parent="robotiq_arg2f_base_link" use_nominal_extrinsics="$(arg use_nominal_extrinsics)">
+    <!-- y + 1.5cm, x + 8cm, pitch - pi/2 -->
+    <origin xyz="0.08 0.0 0.015" rpy="0.0 ${-pi/2} 0.0"/>
+  </xacro:sensor_d455>
   <link name="world" />
   <joint name="world_joint" type="fixed">

Commit message: import table to custom robot xacro

File: workspace/noetic_src/ur_pick_and_place/urdf/ur5/custom_ur5.xacro (robot description, xacro)
@@ -8,4 +8,5 @@
   <!-- import realsense d455 -->
   <xacro:include filename="$(find ur_pick_and_place)/urdf/realsensed455/_d455.urdf.xacro" />
+  <xacro:include filename="$(find ur_pick_and_place)/urdf/ur5/table.urdf.xacro"/>
   <!-- parameters -->
   <!-- ur5 -->
@@ -16,5 +17,6 @@
   <xacro:sensor_d455 parent="robotiq_arg2f_base_link" use_nominal_extrinsics="$(arg use_nominal_extrinsics)">
     <!-- y + 1.5cm, x + 8cm, pitch - pi/2 -->
-    <origin xyz="0.08 0.0 0.015" rpy="0.0 ${-pi/2} 0.0"/>
+    <!-- <origin xyz="0.08 0.0 0.015" rpy="0.0 ${-pi/2} 0.0"/>  -->
+    <origin xyz="0.095 0.0 0.023" rpy="0.0 ${-pi/2} 0.0"/>
   </xacro:sensor_d455>
   <link name="world" />
@@ -29,3 +31,8 @@
     <origin xyz="0 0 0" rpy="0.0 ${pi/2} 0.0"/>
   </joint>
+  <joint name="world_to_table" type="fixed">
+    <parent link="world"/>
+    <child link="table_top_link"/>
+    <origin xyz="0 0 0" rpy="0 0 0"/>
+  </joint>
 </robot>

Commit message: update realsense position on robot custom xacro

File: workspace/noetic_src/ur_pick_and_place/urdf/ur5/custom_ur5.xacro (robot description, xacro)
@@ -18,5 +18,5 @@
     <!-- y + 1.5cm, x + 8cm, pitch - pi/2 -->
     <!-- <origin xyz="0.08 0.0 0.015" rpy="0.0 ${-pi/2} 0.0"/>  -->
-    <origin xyz="0.095 0.0 0.023" rpy="0.0 ${-pi/2} 0.0"/>
+    <origin xyz="0.09 0.0 0.023" rpy="0.0 ${-pi/2} 0.0"/>
   </xacro:sensor_d455>
   <link name="world" />
